File: Phases/Phase-A/KiCAD_Files/Analog_Filtering.kicad_sch (KiCad schematic)
At the start: 25 parts

Commit message: finished filtering
Parts:
- gave numbers to parts that had none: 20
Changed lines of the file:
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@@
 		(dnp no)
 		(fields_autoplaced yes)
-		(property "Reference" "R?"
+		(property "Reference" "R5"
 			(at 101.6 82.55 90)
 			(show_name no)
@@
 			(project "KiCAD_Files"
 				(path "/1a22c328-b2bb-4d71-933f-a069c99db071/3d3b4737-a26d-497e-96ed-58c99ade29b8"
-					(reference "R?")
+					(reference "R5")
 					(unit 1)
 				)
@@
 		(dnp no)
 		(fields_autoplaced yes)
-		(property "Reference" "U?"
+		(property "Reference" "U2"
 			(at 163.83 69.85 0)
 			(show_name no)
@@
 			(project "KiCAD_Files"
 				(path "/1a22c328-b2bb-4d71-933f-a069c99db071/3d3b4737-a26d-497e-96ed-58c99ade29b8"
-					(reference "U?")
+					(reference "U2")
 					(unit 2)
 				)
@@
 		(in_pos_files yes)
 		(dnp no)
-		(property "Reference" "U?"
+		(property "Reference" "U1"
 			(at 86.36 102.362 0)
 			(show_name no)
@@
 			(project "KiCAD_Files"
 				(path "/1a22c328-b2bb-4d71-933f-a069c99db071/3d3b4737-a26d-497e-96ed-58c99ade29b8"
-					(reference "U?")
+					(reference "U1")
 					(unit 2)
 				)
@@
 		(in_pos_files yes)
 		(dnp no)
-		(property "Reference" "R?"
+		(property "Reference" "R11"
 			(at 187.96 74.9299 90)
 			(show_name no)
@@
 			(project "KiCAD_Files"
 				(path "/1a22c328-b2bb-4d71-933f-a069c99db071/3d3b4737-a26d-497e-96ed-58c99ade29b8"
-					(reference "R?")
+					(reference "R11")
 					(unit 1)
 				)
@@
 		(dnp no)
 		(fields_autoplaced yes)
-		(property "Reference" "R?"
+		(property "Reference" "R7"
 			(at 118.11 55.88 90)
 			(show_name no)
@@
 			(project "KiCAD_Files"
 				(path "/1a22c328-b2bb-4d71-933f-a069c99db071/3d3b4737-a26d-497e-96ed-58c99ade29b8"
-					(reference "R?")
+					(reference "R7")
 					(unit 1)
 				)
@@
 		(dnp no)
 		(fields_autoplaced yes)
-		(property "Reference" "C?"
+		(property "Reference" "C2"
 			(at 63.5 91.44 90)
 			(show_name no)
@@
 			(project "KiCAD_Files"
 				(path "/1a22c328-b2bb-4d71-933f-a069c99db071/3d3b4737-a26d-497e-96ed-58c99ade29b8"
-					(reference "C?")
+					(reference "C2")
 					(unit 1)
 				)
@@
 		(dnp no)
 		(fields_autoplaced yes)
-		(property "Reference" "C?"
+		(property "Reference" "C1"
 			(at 63.5 49.53 90)
 			(show_name no)
@@
 			(project "KiCAD_Files"
 				(path "/1a22c328-b2bb-4d71-933f-a069c99db071/3d3b4737-a26d-497e-96ed-58c99ade29b8"
-					(reference "C?")
+					(reference "C1")
 					(unit 1)
 				)
@@
 		(dnp no)
 		(fields_autoplaced yes)
-		(property "Reference" "R?"
+		(property "Reference" "R6"
 			(at 110.49 93.9799 0)
 			(show_name no)
@@
 			(project "KiCAD_Files"
 				(path "/1a22c328-b2bb-4d71-933f-a069c99db071/3d3b4737-a26d-497e-96ed-58c99ade29b8"
-					(reference "R?")
+					(reference "R6")
 					(unit 1)
 				)
@@
 		(dnp no)
 		(fields_autoplaced yes)
-		(property "Reference" "U?"
+		(property "Reference" "U1"
 			(at 86.36 49.53 0)
 			(show_name no)
@@
 			(project "KiCAD_Files"
 				(path "/1a22c328-b2bb-4d71-933f-a069c99db071/3d3b4737-a26d-497e-96ed-58c99ade29b8"
-					(reference "U?")
+					(reference "U1")
 					(unit 1)
 				)
@@
 		(in_pos_files yes)
 		(dnp no)
-		(property "Reference" "C?"
+		(property "Reference" "C5"
 			(at 193.04 88.8999 0)
 			(show_name no)
@@
 			(project "KiCAD_Files"
 				(path "/1a22c328-b2bb-4d71-933f-a069c99db071/3d3b4737-a26d-497e-96ed-58c99ade29b8"
-					(reference "C?")
+					(reference "C5")
 					(unit 1)
 				)
@@
 		(dnp no)
 		(fields_autoplaced yes)
-		(property "Reference" "U?"
+		(property "Reference" "U2"
 			(at 148.59 129.5399 0)
 			(show_name no)
@@
 			(project "KiCAD_Files"
 				(path "/1a22c328-b2bb-4d71-933f-a069c99db071/3d3b4737-a26d-497e-96ed-58c99ade29b8"
-					(reference "U?")
+					(reference "U2")
 					(unit 3)
 				)
@@
 		(in_pos_files yes)
 		(dnp no)
-		(property "Reference" "R?"
+		(property "Reference" "R9"
 			(at 153.67 57.1499 90)
 			(show_name no)
@@
 			(project "KiCAD_Files"
 				(path "/1a22c328-b2bb-4d71-933f-a069c99db071/3d3b4737-a26d-497e-96ed-58c99ade29b8"
-					(reference "R?")
+					(reference "R9")
 					(unit 1)
 				)
@@
 		(dnp no)
 		(fields_autoplaced yes)
-		(property "Reference" "R?"
+		(property "Reference" "R3"
 			(at 86.36 82.55 90)
 			(show_name no)
@@
 			(project "KiCAD_Files"
 				(path "/1a22c328-b2bb-4d71-933f-a069c99db071/3d3b4737-a26d-497e-96ed-58c99ade29b8"
-					(reference "R?")
+					(reference "R3")
 					(unit 1)
 				)
@@
 		(dnp no)
 		(fields_autoplaced yes)
-		(property "Reference" "U?"
+		(property "Reference" "U3"
 			(at 210.82 72.39 0)
 			(show_name no)
@@
 			(project "KiCAD_Files"
 				(path "/1a22c328-b2bb-4d71-933f-a069c99db071/3d3b4737-a26d-497e-96ed-58c99ade29b8"
-					(reference "U?")
+					(reference "U3")
 					(unit 1)
 				)
@@
 		(dnp no)
 		(fields_autoplaced yes)
-		(property "Reference" "C?"
+		(property "Reference" "C3"
 			(at 133.35 69.85 90)
 			(show_name no)
@@
 			(project "KiCAD_Files"
 				(path "/1a22c328-b2bb-4d71-933f-a069c99db071/3d3b4737-a26d-497e-96ed-58c99ade29b8"
-					(reference "C?")
+					(reference "C3")
 					(unit 1)
 				)
@@
 		(dnp no)
 		(fields_autoplaced yes)
-		(property "Reference" "U?"
+		(property "Reference" "U3"
 			(at 165.1 129.5399 0)
 			(show_name no)
@@
 			(project "KiCAD_Files"
 				(path "/1a22c328-b2bb-4d71-933f-a069c99db071/3d3b4737-a26d-497e-96ed-58c99ade29b8"
-					(reference "U?")
+					(reference "U3")
 					(unit 3)
 				)
@@
 		(in_pos_files yes)
 		(dnp no)
-		(property "Reference" "U?"
+		(property "Reference" "U1"
 			(at 132.08 129.5399 0)
 			(show_name no)
@@
 			(project "KiCAD_Files"
 				(path "/1a22c328-b2bb-4d71-933f-a069c99db071/3d3b4737-a26d-497e-96ed-58c99ade29b8"
-					(reference "U?")
+					(reference "U1")
 					(unit 3)
 				)
@@
 		(in_pos_files yes)
 		(dnp no)
-		(property "Reference" "R?"
+		(property "Reference" "R8"
 			(at 148.59 87.6299 0)
 			(show_name no)
@@
 			(project "KiCAD_Files"
 				(path "/1a22c328-b2bb-4d71-933f-a069c99db071/3d3b4737-a26d-497e-96ed-58c99ade29b8"
-					(reference "R?")
+					(reference "R8")
 					(unit 1)
 				)
@@
 		(in_pos_files yes)
 		(dnp no)
-		(property "Reference" "R?"
+		(property "Reference" "R10"
 			(at 177.8 74.9299 90)
 			(show_name no)
@@
 			(project "KiCAD_Files"
 				(path "/1a22c328-b2bb-4d71-933f-a069c99db071/3d3b4737-a26d-497e-96ed-58c99ade29b8"
-					(reference "R?")
+					(reference "R10")
 					(unit 1)
 				)
@@
 		(in_pos_files yes)
 		(dnp no)
-		(property "Reference" "R?"
+		(property "Reference" "R2"
 			(at 86.106 70.866 90)
 			(show_name no)
@@
 			(project "KiCAD_Files"
 				(path "/1a22c328-b2bb-4d71-933f-a069c99db071/3d3b4737-a26d-497e-96ed-58c99ade29b8"
-					(reference "R?")
+					(reference "R2")
 					(unit 1)
 				)
@@
 		(in_pos_files yes)
 		(dnp no)
-		(property "Reference" "R?"
+		(property "Reference" "R1"
 			(at 62.992 76.2 0)
 			(show_name no)
@@
 			(project "KiCAD_Files"
 				(path "/1a22c328-b2bb-4d71-933f-a069c99db071/3d3b4737-a26d-497e-96ed-58c99ade29b8"
-					(reference "R?")
+					(reference "R1")
 					(unit 1)
 				)
@@
 		(dnp no)
 		(fields_autoplaced yes)
-		(property "Reference" "U?"
+		(property "Reference" "U2"
 			(at 119.38 67.31 0)
 			(show_name no)
@@
 			(project "KiCAD_Files"
 				(path "/1a22c328-b2bb-4d71-933f-a069c99db071/3d3b4737-a26d-497e-96ed-58c99ade29b8"
-					(reference "U?")
+					(reference "U2")
 					(unit 1)
 				)
@@
 		(dnp no)
 		(fields_autoplaced yes)
-		(property "Reference" "C?"
+		(property "Reference" "C4"
 			(at 143.51 69.85 90)
 			(show_name no)
@@
 			(project "KiCAD_Files"
 				(path "/1a22c328-b2bb-4d71-933f-a069c99db071/3d3b4737-a26d-497e-96ed-58c99ade29b8"
-					(reference "C?")
+					(reference "C4")
 					(unit 1)
 				)
@@
 		(dnp no)
 		(fields_autoplaced yes)
-		(property "Reference" "R?"
+		(property "Reference" "R4"
 			(at 101.6 60.96 90)
 			(show_name no)
@@
 			(project "KiCAD_Files"
 				(path "/1a22c328-b2bb-4d71-933f-a069c99db071/3d3b4737-a26d-497e-96ed-58c99ade29b8"
-					(reference "R?")
+					(reference "R4")
 					(unit 1)
 				)
@@
 		(in_pos_files yes)
 		(dnp no)
-		(property "Reference" "C?"
+		(property "Reference" "C6"
 			(at 200.66 58.4199 90)
 			(show_name no)
@@
 			(project "KiCAD_Files"
 				(path "/1a22c328-b2bb-4d71-933f-a069c99db071/3d3b4737-a26d-497e-96ed-58c99ade29b8"
-					(reference "C?")
+					(reference "C6")
 					(unit 1)
 				)
