File: Phases/Phase-A/KiCAD_Files/KiCAD_Files.kicad_sch (KiCad schematic)
At the start: 0 parts

Commit message: Analog Filtering Subschematic
Other:
- added sheet Filtering (Analog_Filtering.kicad_sch)
Changed lines of the file:
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@@
 	(generator_version "10.0")
 	(paper "A4")
+	(sheet
+		(at 110.49 92.71)
+		(size 38.1 21.59)
+		(exclude_from_sim no)
+		(in_bom yes)
+		(on_board yes)
+		(dnp no)
+		(fields_autoplaced yes)
+		(stroke
+			(width 0.1524)
+			(type solid)
+			(color 194 0 0 1)
+		)
+		(fill
+			(color 0 0 0 0)
+		)
+		(property "Sheetname" "Filtering"
+			(at 110.49 91.9984 0)
+			(show_name no)
+			(do_not_autoplace no)
+			(effects
+				(font
+					(size 1.27 1.27)
+				)
+				(justify left bottom)
+			)
+		)
+		(property "Sheetfile" "Analog_Filtering.kicad_sch"
+			(at 110.49 114.8846 0)
+			(show_name no)
+			(do_not_autoplace no)
+			(effects
+				(font
+					(size 1.27 1.27)
+				)
+				(justify left top)
+			)
+		)
+		(instances
+			(project "KiCAD_Files"
+				(path "/1a22c328-b2bb-4d71-933f-a069c99db071"
+					(page "2")
+				)
+			)
+		)
+	)
 	(sheet_instances
 		(path "/"

Commit message: finished filtering
Parts:
- added J?: USB_C_Receptacle_USB2.0_14P, symbol Connector:USB_C_Receptacle_USB2.0_14P
- added R? (x2): R, symbol Device:R
Connections:
- new net: J?.A5 (CC1), R?.1
- new net: J?.A6 (D+), J?.B6 (D+)
- new net: J?.A7 (D-), J?.B7 (D-)
- new net: J?.B5 (CC2), R?.1
- new net +5V: J?.A4 (VBUS), J?.A9 (VBUS), J?.B4 (VBUS), J?.B9 (VBUS)
- new net GND: J?.A1 (GND), J?.A12 (GND), J?.B1 (GND), J?.B12 (GND), R?.2, R?.2
- no-connect marks 0 -> 1

Commit message: Added Filtering + ECG Circuit to Sch
Parts:
- added C1, C10, C11, C12, C2, C3, C4, C5, C6, C7, C8, C9: ${ALTIUM_VALUE}, CAPC1608X06L, symbol AltiumLib:CAP
- added C13: ${ALTIUM_VALUE}, CAPC0603X03L_C, symbol AltiumLib:CAP
- added C? (x4): 2.2u, symbol Device:C
- added C? (x4): 1u, symbol Device:C
- added C? (x4): 100n, symbol Device:C
- added C?: 10u, symbol Device:C
- added C?: 150n, symbol Device:C
- added C?: 10n, symbol Device:C
- added FB?: FerriteBead, symbol Device:FerriteBead
- added J1: ${ALTIUM_VALUE}, TP_3x1mm_TH, symbol AltiumLib:Battery_pack_NTC
- added L1, L2: ${ALTIUM_VALUE}, INDC2016X10N, symbol AltiumLib:IND
- added L?: 4.7u, symbol Device:L
- added LD1: ${ALTIUM_VALUE}, LED_RGB_0603, symbol AltiumLib:D{colon}LED_RGB
- added NT1, NT2: ${ALTIUM_VALUE}, 2 PIN STARPOINT, symbol AltiumLib:2 pin starpoint
- added R1, R2, R3, R4: ${ALTIUM_VALUE}, RESC0603X03L_C, symbol AltiumLib:RES
- added R? (x2): 330k, symbol Device:R
- added R? (x2): 5k, symbol Device:R
- added R?: 220k, symbol Device:R
- added R?: 560k, symbol Device:R
- added R? (x2): 2k, symbol Device:R
- added R?: 18k, symbol Device:R
- added R?: 120k, symbol Device:R
- added R?: R_Variable, symbol Device:R_Variable
- added U1: ${ALTIUM_VALUE}, Nordic_QFN50P500X500X90-33N, symbol AltiumLib:nPM1300_QEAA
- added U? (x8): Opamp_Dual, symbol Amplifier_Operational:Opamp_Dual
- added U?: nRF54L15-QFXX, Package_DFN_QFN:QFN-48-1EP_6x6mm_P0.4mm_EP4.6x4.6mm_ThermalVias, symbol nordic-lib-kicad-nrf54l:nRF54L15-QFXX
- added Y?: Crystal_GND3, symbol Device:Crystal_GND3
Connections:
- net GND: now also C1.1, C10.1, C11.1, C12.1, C13.2, C4.1, C5.1, C6.1, C9.1, C?.2, C?.2, C?.2, C?.2, C?.2, C?.2, C?.2, C?.2, C?.2, J1.1 (GND), NT1.1, NT2.1, R3.2, R4.2, U1.33 (AVSS), U?.4 (V-), U?.4 (V-), U?.8 (V+)
- new net: C?.1, C?.2, R?.2
- new net: C?.2, R?.2, U?.5 (+)
- new net: R?.1, R?.2, U?.2 (-)
- new net: C?.1, R?.2, U?.1
- new net: R?.1, R?.1, U?.2 (-)
- new net: R?.1, R?.2, U?.1
- new net: C?.2, R?.1, U?.3 (+)
- new net: R?.1, R?.2, U?.6 (-)
- new net: R?.1, R?.2, U?.7
- new net: R?.2, R?.2, U?.3 (+)
- new net: C?.2, R?.1, R?.2
- new net: U?.34 (XC1), Y?.1
- new net: U?.35 (XC2), Y?.3
- new net: R?.1, R?.2, U?.6 (-), U?.7
- new net: U?.22 (VDD), U?.36 (VDD), U?.47 (VDD), U?.48 (VDD)
- new net: U?.32 (VSS_PA), U?.44 (VSS), U?.49 (VSS)
- new net +3V3: C?.1, C?.1, C?.1, C?.1, C?.1, U?.47 (VDD), U?.48 (VDD)
- new net ANT: U?.31 (ANT)
- new net CC1: U1.23 (CC1)
- new net CC2: U1.24 (CC2)
- new net DCC: L?.1, U?.46 (DCC)
- new net DEC_A: C?.1, C?.1, C?.1, FB?.1, U?.33 (DECRF), U?.43 (DECA)
- new net DEC_D: C?.1, FB?.2, L?.2, U?.45 (DECD)
- new net ECG_OUT: C?.1, U?.1, U?.2 (-)
- new net GPIO0: U1.7 (GPIO0)
- new net GPIO1: U1.8 (GPIO1)
- new net GPIO2: U1.9 (GPIO2)
- new net GPIO3: U1.10 (GPIO3)
- new net GPIO4: U1.11 (GPIO4)
- new net LED0: LD1.3 (C_BLUE), U1.25 (LED0)
- new net LED1: LD1.2 (C_GREEN), U1.26 (LED1)
- new net LED2: LD1.1 (C_RED), U1.27 (LED2)
- new net NTC: J1.2 (NTC), U1.18 (NTC)
- new net POWER: U?.4 (V-), U?.8 (V+), U?.8 (V+)
- new net PVSS1: C2.1, C7.1, NT1.2, U1.2 (PVSS1)
- new net PVSS2: C3.1, C8.1, NT2.2, U1.6 (PVSS2)
- new net RST: U?.30 (~{RESET})
- new net SCL: R1.1, U1.14 (SCL)
- new net SDA: R2.1, U1.13 (SDA)
- new net SHPHLD: U1.15 (SHPHLD)
- new net SW1: L1.2, U1.3 (SW1)
- new net SW2: L2.2, U1.5 (SW2)
- new net SWD0_SWDCLK: U?.26 (SWDCLK)
- new net SWD0_SWDIO: U?.25 (SWDIO)
- new net VBAT: C6.2, J1.3 (V+), U1.19 (VBAT)
- new net VBUSIN: C1.2, U1.21 (VBUS)
- new net VBUSOUT: C5.2, U1.22 (VBUSOUT)
- new net VDDIO: C13.1, R1.2, R2.2, U1.12 (VDDIO)
- new net VDD_FILL_1: U?.10 (VDD), U?.22 (VDD), U?.36 (VDD)
- new net VINLDO1: U1.28 (LSIN1/VINLDO1)
- new net VINLDO2: U1.30 (LSIN2/VINLDO2)
- new net VOUT1: C7.2, L1.1, U1.1 (VOUT1)
- new net VOUT2: C8.2, L2.1, U1.32 (VOUT2)
- new net VOUTLDO1: C10.2, C9.2, U1.29 (LSOUT1/VOUTLDO1)
- new net VOUTLDO2: C11.2, C12.2, U1.31 (LSOUT2/VOUTLDO2)
- new net VSET1: R3.1, U1.17 (VSET1)
- new net VSET2: R4.1, U1.16 (VSET2)
- new net VSYS: C2.2, C3.2, C4.2, LD1.4 (A), U1.20 (VSYS), U1.4 (PVDD)
- new net bias: C?.1, C?.2, C?.2, R?.1, R?.1, U?.3 (+), U?.5 (+)
- no-connect marks 1 -> 6
Other:
- removed sheet Filtering
- note added: "1.8 V"
- note added: "3.0 V"
- note added: "ECG CIRCUIT"
- note added: "FILTERING"
- note added: "Via to GND-layer on PVSS1"
- note added: "Via to GND-layer on PVSS2"

Commit message: Fleshed out PMIC wiring based off i2cjak vid
Parts:
- removed C? (x4): 2.2u, symbol Device:C
- removed C? (x4): 100n, symbol Device:C
- removed C?: 10u, symbol Device:C
- removed FB?: FerriteBead, symbol Device:FerriteBead
- removed J?: USB_C_Receptacle_USB2.0_14P, symbol Connector:USB_C_Receptacle_USB2.0_14P
- removed L?: 4.7u, symbol Device:L
- removed R? (x2): R, symbol Device:R
- removed U?: nRF54L15-QFXX, Package_DFN_QFN:QFN-48-1EP_6x6mm_P0.4mm_EP4.6x4.6mm_ThermalVias, symbol nordic-lib-kicad-nrf54l:nRF54L15-QFXX
- removed Y?: Crystal_GND3, symbol Device:Crystal_GND3
- added C? (x9): 10uF, symbol Device:C
- added C?: 100nF, symbol Device:C
- added C? (x2): 1uF, symbol Device:C
- added C?: 2.2uF, symbol Device:C
- added D?: LED_ARGB, symbol Device:LED_ARGB
- added F?: Polyfuse, symbol Device:Polyfuse
- added J?: USB_C_Receptacle_PowerOnly_6P, symbol Connector:USB_C_Receptacle_PowerOnly_6P
- added J?: Conn_01x02_MountingPin, symbol Connector_Generic_MountingPin:Conn_01x02_MountingPin
- added L? (x2): ${ALTIUM_VALUE}, INDC2016X10N, symbol AltiumLib:IND
- added U?: nPM1300-QEXX, Package_DFN_QFN:QFN-32-1EP_5x5mm_P0.5mm_EP3.6x3.6mm_ThermalVias, symbol PCM_nordic-lib-kicad-npm:nPM1300-QEXX
Connections:
- net GND: now also C?.2, C?.2, C?.2, C?.2, C?.2, C?.2, C?.2, C?.2, C?.2, C?.2, C?.2, C?.2, C?.2, J?.2 (Pin_2), J?.MP (MountPin), U?.2 (PVSS1), U?.6 (PVSS2)
- net VSYS: now also C?.1, C?.1, C?.1, D?.1 (A), U?.20 (VSYS), U?.4 (PVDD)
- new net: C?.1, C?.1, U?.29 (LSOUT1/VOUTLDO1)
- new net: C?.1, L?.1, U?.32 (VOUT2)
- new net: L?.2, U?.5 (SW2)
- new net: F?.1, J?.A9 (VBUS), J?.B9 (VBUS)
- new net: C?.1, F?.2, U?.21 (VBUS)
- new net: C?.1, U?.12 (VDDIO)
- new net: C?.1, L?.1, U?.1 (VOUT1)
- new net: C?.1, J?.1 (Pin_1), U?.19 (VBAT)
- new net: C?.1, U?.22 (VBUSOUT)
- new net: D?.2 (RK), U?.25 (LED0)
- new net: D?.3 (GK), U?.26 (LED1)
- new net: D?.4 (BK), U?.27 (LED2)
- new net: L?.2, U?.3 (SW1)
- new net: C?.1, C?.1, U?.31 (LSOUT2/VOUTLDO2)
- new net: J?.A12 (GND), J?.B12 (GND)
- no-connect marks 6 -> 0
Other:
- note removed: "FILTERING"
- moved on the sheet: C1, C10, C11, C12, C13, C2, C3, C4, C5, C6, C7, C8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
